File: ultra-low-pcb/ultra-low-pcb.kicad_pcb (KiCad board)
At the start: 2 copper layers, 77.9 x 45.2 mm, 39 parts, among them IC1 ESP32-C3-WROOM-02-N4, IC2 TPS2117DRLR, J1 USB_C_Receptacle_USB2.0, J2 S2B-PH-SM4-TB_LF__SN_, J3 FH52-10S-0.5SH_99, Q1 AO3401A, SW1 TC-0522C-1.7-160G, SW2 TC-0522C-1.7-160G, SW3 TC-0522C-1.7-160G, SW4 TC-0522C-1.7-160G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

Commit message: Update U3
Parts:
- added R13: 0Ω, Resistor_SMD:R_0603_1608Metric, F.Cu at (131.7, 91.5)
- R11: value 5.1k -> 10k
- moved R11 2.50 mm to (133.7, 91.9), turned to -135 degrees
Connections:
- R11 pad 2: Net-(Q1-S) -> GND
Routing:
- net Net-(D1-K): track 3.72 -> 7.98 mm
- net MCU_PWRHOLD: track 40.5 -> 43.3 mm
- net GND: track 62.2 -> 62.9 mm, vias 28 -> 29

Commit message: Correct Q1. Thanks Syl!
Parts:
- added R14: r=0, Resistor_SMD:R_0603_1608Metric, F.Cu at (170.6, 101.0)
Connections:
- Q1 pad 2: Net-(Q1-S) -> VIN
- Q1 pad 3: VIN -> Net-(Q1-D)
- R13 pad 1: Net-(Q1-S) -> Net-(Q1-D)
- R7 pad 2: +3.3V -> +3.3VP
Routing:
- net +3.3V: track 182.4 -> 81.6 mm
- net +3.3VP: track 99.0 -> 105.1 mm
- net Net-(Q1-D): track 0.00 -> 3.19 mm
- net Net-(Q1-S): track 1.93 -> 0.00 mm
- net RTC_EVI: track 31.5 -> 29.8 mm
- net VIN: track 100.5 -> 99.3 mm

Commit message: Put some love in silk
Parts:
- moved D1 0.89 mm to (136.3, 92.2)
Routing:
- net MCU_PWRHOLD: track 43.3 -> 42.6 mm
Other:
- outline, holes or cut-outs redrawn
- board text added: "3V3P keeps only RTC & LCD on"
- board text added: "LowPow"
- board text added: "RTCINT Wake up"
- board text added: "TPS2117"
- board text added: "USB always on"
- board text added: "experi"
- board text added: "ment"
- board text added: "▲SHARP LCD▲"

Commit message: Last revision before 1.0
Parts:
- added J4: Conn_01x02_Socket, Connector_PinHeader_2.54mm:PinHeader_1x02_P2.54mm_Vertical, F.Cu at (181.8, 91.5)
- added R15: 10K, Resistor_SMD:R_0603_1608Metric, F.Cu at (153.7, 95.7)
- added TP1: U3EN, TestPoint:TestPoint_Pad_D1.5mm, F.Cu at (135.4, 88.5)
- added TP2: U4EN, TestPoint:TestPoint_Pad_D1.5mm, F.Cu at (135.4, 97.5)
Connections:
- IC1 pad 7: /IO8 -> PWR_STAT
- Q1 pad 2: VIN -> +3.3VP
Routing:
- net VIN: track 99.3 -> 53.1 mm
- net /RX: track 0.00 -> 24.9 mm
- net /TX: track 0.00 -> 21.8 mm
- net PWR_STAT: track 41.5 -> 61.1 mm
- net +3.3VP: track 105.1 -> 118.8 mm
- net +5V: track 28.5 -> 41.9 mm
- net Net-(D1-K): track 7.60 -> 12.2 mm, vias 0 -> 2
Other:
- outline, holes or cut-outs redrawn
- board text added: "2117 STAT"
- board text added: "Fabrication costs sponsored by HELENA CORP. fundation"
- board text added: "RX"
- board text added: "TX"
- board text added: "U3EN"
- board text added: "U4EN"
- board text added: "▲pull-up"
