File: ultra-low-pcb/ultra-low-pcb.kicad_sch (KiCad schematic)
At the start: 41 parts, among them IC1 ESP32-C3-WROOM-02-N4, IC2 TPS2117DRLR, J1 USB_C_Receptacle_USB2.0, J2 S2B-PH-SM4-TB_LF__SN_, J3 FH52-10S-0.5SH_99, Q1 AO3401A, SW1 TC-0522C-1.7-160G, SW2 TC-0522C-1.7-160G, SW3 TC-0522C-1.7-160G, SW4 TC-0522C-1.7-160G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

Commit message: Last revision before 1.0
Parts:
- added J4: Conn_01x02_Socket, Connector_PinHeader_2.54mm:PinHeader_1x02_P2.54mm_Vertical, symbol Connector:Conn_01x02_Socket
- added R15: 10K, Resistor_SMD:R_0603_1608Metric, symbol Device:R
- added TP1: U3EN, TestPoint:TestPoint_Pad_D1.5mm, symbol Connector:TestPoint
- added TP2: U4EN, TestPoint:TestPoint_Pad_D1.5mm, symbol Connector:TestPoint
Connections:
- net IO8 is gone; now on net PWR_STAT: IC1.7 (IO8)
- net +3.3VP: now also Q1.2 (S), R15.2
- net PWR_STAT: now also R15.1, TP2.1
- net RX: now also J4.1 (Pin_1)
- net TX: now also J4.2 (Pin_2)
- net VIN: no longer Q1.2 (S)
- net at D1.1 (K), R11.1, R13.2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: now also TP1.1
Other:
- moved on the sheet: C1, C2, U2
