File: ultra-low-pcb/ultra-low-pcb.kicad_sch (KiCad schematic)
At the start: 45 parts, among them IC1 ESP32-C3-WROOM-02-N4, IC2 TPS2117DRLR, J1 USB_C_Receptacle_USB2.0, J2 S2B-PH-SM4-TB_LF__SN_, J3 FH52-10S-0.5SH_99, J4 Conn_01x02_Socket, Q1 AO3401A, SW1 TC-0522C-1.7-160G, SW2 TC-0522C-1.7-160G, SW3 TC-0522C-1.7-160G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

Commit message: Update SCH
Parts:
- IC1: LCSC (none) -> C2934560; Manufacturer_Part_Number ESP32-C3-WROOM-02-N4 -> (none); Mouser Part Number 356-ESP32C3WROOM02N4 -> (none); Mouser Price/Stock https://www.mouser.co.uk/ProductDetail/Espressif-Systems/ES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 -> (none)
Other:
- note added: "MAIN LDO powers MCU"
- note added: "Small LDO only RTC & LCD"
- moved on the sheet: C1, C2, C7, C8, SW3, TP2, U2, U4, U6
